Commit message: fix bug

File: robot/mobile_bot/urdf/mobile_bot.urdf (robot description, URDF)
Before this commit: robot mobile_bot, 5 links, 4 joints
Joints:
- joint camera_joint: origin xyz=.35 0 .25 rpy=0 0.8 0 -> xyz=.35 0 .20 rpy=0 0.7 0

Commit message: fix car rolling

File: robot/mobile_bot/urdf/mobile_bot.urdf (robot description, URDF)
Before this commit: robot mobile_bot, 5 links, 4 joints
Links:
- link aux_link: geometry collision cylinder length=0.05 radius=0.039; visual mesh filename=package://mobile_bot/meshes/aux_link.STL
- link left_wheel_link: geometry collision cylinder length=0.05 radius=0.1; visual mesh filename=package://mobile_bot/meshes/left_wheel_link.STL
- link right_wheel_link: geometry collision cylinder length=0.05 radius=0.1; visual mesh filename=package://mobile_bot/meshes/right_wheel_link.STL
